Commit message: Updated the m6ib6s_support and implemented it inside m6ib_support

File: fanuc/fanuc_m6ib_support/urdf/m6ib6s.xacro (robot description, xacro)
@@ -1,5 +1,5 @@
 <?xml version="1.0"?>
 <robot name="fanuc_m6ib6s" xmlns:xacro="http://wiki.ros.org/xacro">
-  <xacro:include filename="$(find fanuc_m6ib6s_support)/urdf/m6ib6s_macro.xacro"/>
+  <xacro:include filename="$(find fanuc_m6ib_support)/urdf/m6ib6s_macro.xacro"/>
   <xacro:fanuc_m6ib6s prefix=""/>
 </robot>

File: fanuc/fanuc_m6ib_support/urdf/m6ib6s_macro.xacro (robot description, xacro)
@@ -8,5 +8,5 @@
         <origin xyz="0 0 0" rpy="0 0 0"/>
         <geometry>
-          <mesh filename="package://fanuc_m6ib6s_support/meshes/m6ib6s/visual/base_link.stl"/>
+          <mesh filename="package://fanuc_m6ib_support/meshes/m6ib6s/visual/base_link.stl"/>
         </geometry>
         <xacro:material_fanuc_grey />
@@ -15,5 +15,5 @@
         <origin xyz="0 0 0" rpy="0 0 0"/>
         <geometry>
-          <mesh filename="package://fanuc_m6ib6s_support/meshes/m6ib6s/collision/base_link.stl"/>
+          <mesh filename="package://fanuc_m6ib_support/meshes/m6ib6s/collision/base_link.stl"/>
         </geometry>
       </collision>
@@ -23,5 +23,5 @@
         <origin xyz="0 0 0" rpy="0 0 0"/>
         <geometry>
-          <mesh filename="package://fanuc_m6ib6s_support/meshes/m6ib6s/visual/link_1.stl"/>
+          <mesh filename="package://fanuc_m6ib_support/meshes/m6ib6s/visual/link_1.stl"/>
         </geometry>
         <xacro:material_fanuc_yellow />
@@ -30,5 +30,5 @@
         <origin xyz="0 0 0" rpy="0 0 0"/>
         <geometry>
-          <mesh filename="package://fanuc_m6ib6s_support/meshes/m6ib6s/collision/link_1.stl"/>
+          <mesh filename="package://fanuc_m6ib_support/meshes/m6ib6s/collision/link_1.stl"/>
         </geometry>
       </collision>
@@ -38,5 +38,5 @@
         <origin xyz="0 0 0" rpy="0 0 0"/>
         <geometry>
-          <mesh filename="package://fanuc_m6ib6s_support/meshes/m6ib6s/visual/link_2.stl"/>
+          <mesh filename="package://fanuc_m6ib_support/meshes/m6ib6s/visual/link_2.stl"/>
         </geometry>
         <xacro:material_fanuc_yellow />
@@ -45,5 +45,5 @@
         <origin xyz="0 0 0" rpy="0 0 0"/>
         <geometry>
-          <mesh filename="package://fanuc_m6ib6s_support/meshes/m6ib6s/collision/link_2.stl"/>
+          <mesh filename="package://fanuc_m6ib_support/meshes/m6ib6s/collision/link_2.stl"/>
         </geometry>
       </collision>
@@ -53,5 +53,5 @@
         <origin xyz="0 0 0" rpy="0 0 0"/>
         <geometry>
-          <mesh filename="package://fanuc_m6ib6s_support/meshes/m6ib6s/visual/link_3.stl"/>
+          <mesh filename="package://fanuc_m6ib_support/meshes/m6ib6s/visual/link_3.stl"/>
         </geometry>
         <xacro:material_fanuc_yellow />
@@ -60,5 +60,5 @@
         <origin xyz="0 0 0" rpy="0 0 0"/>
         <geometry>
-          <mesh filename="package://fanuc_m6ib6s_support/meshes/m6ib6s/collision/link_3.stl"/>
+          <mesh filename="package://fanuc_m6ib_support/meshes/m6ib6s/collision/link_3.stl"/>
         </geometry>
       </collision>
@@ -68,5 +68,5 @@
         <origin xyz="0 0 0" rpy="0 0 0"/>
         <geometry>
-          <mesh filename="package://fanuc_m6ib6s_support/meshes/m6ib6s/visual/link_4.stl"/>
+          <mesh filename="package://fanuc_m6ib_support/meshes/m6ib6s/visual/link_4.stl"/>
         </geometry>
         <xacro:material_fanuc_yellow />
@@ -75,5 +75,5 @@
         <origin xyz="0 0 0" rpy="0 0 0"/>
         <geometry>
-          <mesh filename="package://fanuc_m6ib6s_support/meshes/m6ib6s/collision/link_4.stl"/>
+          <mesh filename="package://fanuc_m6ib_support/meshes/m6ib6s/collision/link_4.stl"/>
         </geometry>
       </collision>
@@ -83,5 +83,5 @@
         <origin xyz="0 0 0" rpy="0 0 0"/>
         <geometry>
-          <mesh filename="package://fanuc_m6ib6s_support/meshes/m6ib6s/visual/link_5.stl"/>
+          <mesh filename="package://fanuc_m6ib_support/meshes/m6ib6s/visual/link_5.stl"/>
         </geometry>
         <xacro:material_fanuc_yellow />
@@ -90,5 +90,5 @@
         <origin xyz="0 0 0" rpy="0 0 0"/>
         <geometry>
-          <mesh filename="package://fanuc_m6ib6s_support/meshes/m6ib6s/collision/link_5.stl"/>
+          <mesh filename="package://fanuc_m6ib_support/meshes/m6ib6s/collision/link_5.stl"/>
         </geometry>
       </collision>
@@ -98,5 +98,5 @@
         <origin xyz="0 0 0" rpy="0 0 0"/>
         <geometry>
-          <mesh filename="package://fanuc_m6ib6s_support/meshes/m6ib6s/visual/link_6.stl"/>
+          <mesh filename="package://fanuc_m6ib_support/meshes/m6ib6s/visual/link_6.stl"/>
         </geometry>
         <xacro:material_fanuc_black />
@@ -105,5 +105,5 @@
         <origin xyz="0 0 0" rpy="0 0 0"/>
         <geometry>
-          <mesh filename="package://fanuc_m6ib6s_support/meshes/m6ib6s/collision/link_6.stl"/>
+          <mesh filename="package://fanuc_m6ib_support/meshes/m6ib6s/collision/link_6.stl"/>
         </geometry>
       </collision>
