Commit message: before testing parelization

File: smobex_description/urdf/m6ib6s_macro_restricted.xacro (robot description, xacro)
@@ -109,5 +109,5 @@
       </collision>
     </link>
-    <xacro:property name="delta" value="0.1" />
+    <xacro:property name="delta" value="0.2" />
     <!-- joints: main serial chain -->
     <joint name="${prefix}joint_1" type="revolute">

Commit message: small tries

File: smobex_description/urdf/m6ib6s_macro_restricted.xacro (robot description, xacro)
@@ -109,5 +109,5 @@
       </collision>
     </link>
-    <xacro:property name="delta" value="0.2" />
+    <xacro:property name="delta" value="0.0" />
     <!-- joints: main serial chain -->
     <joint name="${prefix}joint_1" type="revolute">
@@ -153,5 +153,6 @@
       <child link="${prefix}link_6"/>
       <axis xyz="-1 0 0"/>
-      <limit lower="${-6.2831+delta}" upper="${6.2831-delta}" effort="0" velocity="12.5663"/>
+      <!-- <limit lower="${-6.2831+delta}" upper="${6.2831-delta}" effort="0" velocity="12.5663"/> -->
+      <limit lower="${-3.14159+delta}" upper="${3.14159-delta}" effort="0" velocity="12.5663"/>
     </joint>
     <!-- ROS-Industrial 'base' frame: base_link to Fanuc World Coordinates transform -->
