Commit message: Added robot pedestal urdf

File: smobex_description/urdf/calibrated.xacro (robot description, xacro)
@@ -14,3 +14,9 @@
         <child link="camera_link"/>
     </joint>
+    <xacro:include filename="$(find pedestal_description)/urdf/pedestal.urdf"/>
+    <joint name="pedestal_joint" type="fixed">
+        <origin xyz="0.00000 0.00000 0.00000" rpy="-3.14159265359 0.00000 0.00000"/>
+        <parent link="base_link"/>
+        <child link="pedestal_description"/>
+    </joint>
 </robot>

Commit message: further limitation of joint bounds

File: smobex_description/urdf/calibrated.xacro (robot description, xacro)
@@ -2,5 +2,5 @@
 <robot xmlns:xacro="http://www.ros.org/wiki/xacro" name="fanuc_xtion">
     <xacro:include filename="$(find smobex_calibration)/calibration/calib_vals.xacro"/>
-    <xacro:include filename="$(find fanuc_m6ib_support)/urdf/m6ib6s_macro.xacro"/>
+    <xacro:include filename="$(find smobex_description)/urdf/m6ib6s_macro_restricted.xacro"/>
     <xacro:fanuc_m6ib6s prefix=""/>
     <xacro:include filename="$(find hector_sensors_description)/urdf/asus_camera.urdf.xacro"/>
@@ -14,5 +14,5 @@
         <child link="camera_link"/>
     </joint>
-    <xacro:include filename="$(find pedestal_description)/urdf/pedestal.urdf"/>
+    <xacro:include filename="$(find smobex_description)/urdf/pedestal.urdf"/>
     <joint name="pedestal_joint" type="fixed">
         <origin xyz="0.00000 0.00000 0.00000" rpy="-3.14159265359 0.00000 0.00000"/>

File: smobex_description/urdf/pedestal.urdf (robot description, URDF)
Before this commit: robot pedestal, 1 links, 0 joints
Links:
- link pedestal_description: geometry collision mesh filename=package://smobex_description/meshes/pedestal_description.STL; visual mesh filename=package://smobex_description/meshes/pedestal_description.STL

Commit message: updates to description

File: smobex_description/urdf/calibrated.xacro (robot description, xacro)
@@ -2,16 +2,20 @@
 <robot xmlns:xacro="http://www.ros.org/wiki/xacro" name="fanuc_xtion">
     <xacro:include filename="$(find smobex_calibration)/calibration/calib_vals.xacro"/>
-    <xacro:include filename="$(find smobex_description)/urdf/m6ib6s_macro_restricted.xacro"/>
+    <xacro:include filename="$(find fanuc_m6ib_support)/urdf/m6ib6s_macro.xacro"/>
+    <!-- <xacro:include filename="$(find smobex_description)/urdf/m6ib6s_macro_restricted.xacro"/> -->
     <xacro:fanuc_m6ib6s prefix=""/>
+    <!-- <xacro:include filename="$(find hector_sensors_description)/urdf/asus_camera.urdf.xacro"/>
+    <xacro:asus_camera_model name="camera" parent="flange">
+        <origin rpy="0 0 0" xyz="0 0 0"/>
+    </xacro:asus_camera_model> -->
+    <!-- <joint name="camera_xtion_joint" type="fixed">
+        <origin rpy="${roll} ${pitch} ${yaw}" xyz="${x} ${y} ${z}"/>
+        <parent link="flange"/>
+        <child link="camera_link"/>
+    </joint> -->
     <xacro:include filename="$(find hector_sensors_description)/urdf/asus_camera.urdf.xacro"/>
     <xacro:asus_camera_model name="camera" parent="flange">
-        <origin rpy="0 0 0" xyz="0 0 0"/>
+        <origin rpy="${roll} ${pitch} ${yaw}" xyz="${x} ${y} ${z}"/>
     </xacro:asus_camera_model>
-    <joint name="camera_xtion_joint" type="fixed">
-        <origin rpy="${roll} ${pitch} ${yaw}" xyz="${x} ${y} ${z}"/>
-        <!-- <origin xyz="1.00000 1.00000 1.00000" rpy="0.00000 0.00000 0.00000"/> -->
-        <parent link="flange"/>
-        <child link="camera_link"/>
-    </joint>
     <xacro:include filename="$(find smobex_description)/urdf/pedestal.urdf"/>
     <joint name="pedestal_joint" type="fixed">

Commit message: pre IKFAST plugin

File: smobex_description/urdf/calibrated.xacro (robot description, xacro)
@@ -20,5 +20,5 @@
     <xacro:include filename="$(find smobex_description)/urdf/pedestal.urdf"/>
     <joint name="pedestal_joint" type="fixed">
-        <origin xyz="0.00000 0.00000 0.00000" rpy="-3.14159265359 0.00000 0.00000"/>
+        <origin xyz="0 0 0" rpy="0 0 0"/>
         <parent link="base_link"/>
         <child link="pedestal_description"/>
