Commit message: Updated params in calibration mode, not working yet

File: smobex_calibration/calibration/calib_vals.xacro (robot description, xacro)
@@ -2,11 +2,11 @@
 <robot xmlns:xacro="http://www.ros.org/wiki/xacro">
 <!--This xacro contains six xacro propperties representing a transformation obtained through calibration-->
-<!--Calibration generated at 11:25:03, 14/03/2019 -->
+<!--Calibration generated at 17:14:18, 14/03/2019 -->
 <!--This file was written automatically using the "rosrun smobex_calibration store_calibration" command. -->
-<xacro:property name="roll" value="-0.00582417085643"/>
-<xacro:property name="pitch" value="0.0603078351675"/>
-<xacro:property name="yaw" value="0.00641184347465"/>
-<xacro:property name="x" value="0.020734392867"/>
-<xacro:property name="y" value="0.0501239963471"/>
-<xacro:property name="z" value="0.0426099532389"/>
+<xacro:property name="roll" value="-0.00506339850584"/>
+<xacro:property name="pitch" value="0.0539262905258"/>
+<xacro:property name="yaw" value="0.0311886770651"/>
+<xacro:property name="x" value="0.0671880576021"/>
+<xacro:property name="y" value="0.0492599859315"/>
+<xacro:property name="z" value="-0.00507698144663"/>
 </robot>

Commit message: Corrected first error,  calibrated robot and camero only had same name

File: smobex_calibration/calibration/calib_vals.xacro (robot description, xacro)
@@ -4,9 +4,9 @@
 <!--Calibration generated at 17:14:18, 14/03/2019 -->
 <!--This file was written automatically using the "rosrun smobex_calibration store_calibration" command. -->
-<xacro:property name="roll" value="-0.00506339850584"/>
-<xacro:property name="pitch" value="0.0539262905258"/>
-<xacro:property name="yaw" value="0.0311886770651"/>
-<xacro:property name="x" value="0.0671880576021"/>
-<xacro:property name="y" value="0.0492599859315"/>
-<xacro:property name="z" value="-0.00507698144663"/>
+<xacro:property name="roll" value="-0.00"/>
+<xacro:property name="pitch" value="0.00"/>
+<xacro:property name="yaw" value="0.00"/>
+<xacro:property name="x" value="0.00"/>
+<xacro:property name="y" value="0.00"/>
+<xacro:property name="z" value="0.00"/>
 </robot>

File: smobex_description/urdf/xtion.xacro (robot description, xacro)
@@ -1,4 +1,4 @@
 <?xml version="1.0"?>
-<robot xmlns:xacro="http://www.ros.org/wiki/xacro" name="fanuc_xtion">
+<robot xmlns:xacro="http://www.ros.org/wiki/xacro" name="xtion">
     <link name="flange" />
     <xacro:include filename="$(find hector_sensors_description)/urdf/asus_camera.urdf.xacro"/>

Commit message: Calibration working fine for the first time

File: smobex_calibration/calibration/calib_vals.xacro (robot description, xacro)
@@ -2,11 +2,11 @@
 <robot xmlns:xacro="http://www.ros.org/wiki/xacro">
 <!--This xacro contains six xacro propperties representing a transformation obtained through calibration-->
-<!--Calibration generated at 17:14:18, 14/03/2019 -->
+<!--Calibration generated at 19:17:24, 15/03/2019 -->
 <!--This file was written automatically using the "rosrun smobex_calibration store_calibration" command. -->
-<xacro:property name="roll" value="-0.00"/>
-<xacro:property name="pitch" value="0.00"/>
-<xacro:property name="yaw" value="0.00"/>
-<xacro:property name="x" value="0.00"/>
-<xacro:property name="y" value="0.00"/>
-<xacro:property name="z" value="0.00"/>
+<xacro:property name="roll" value="0.00934253096996"/>
+<xacro:property name="pitch" value="0.066844248775"/>
+<xacro:property name="yaw" value="0.0175544265835"/>
+<xacro:property name="x" value="0.0898634033575"/>
+<xacro:property name="y" value="0.0386030299782"/>
+<xacro:property name="z" value="-0.00850057584549"/>
 </robot>

File: smobex_description/urdf/xtion.xacro (robot description, xacro)
@@ -1,7 +1,10 @@
 <?xml version="1.0"?>
 <robot xmlns:xacro="http://www.ros.org/wiki/xacro" name="xtion">
-    <link name="flange" />
+    <!-- Created because it was needed a parent -->
+    <link name="cam_flange">
+        <origin xyz="0 0 0" rpy="0 0 0" />
+    </link>
     <xacro:include filename="$(find hector_sensors_description)/urdf/asus_camera.urdf.xacro"/>
-    <xacro:asus_camera_model name="camera" parent="flange">
+    <xacro:asus_camera_model name="camera" parent="cam_flange">
         <origin rpy="0 0 0" xyz="0 0 0"/>
     </xacro:asus_camera_model>

Commit message: Update to readme. Added video of the calibration process

File: smobex_calibration/calibration/calib_vals.xacro (robot description, xacro)
@@ -2,11 +2,11 @@
 <robot xmlns:xacro="http://www.ros.org/wiki/xacro">
 <!--This xacro contains six xacro propperties representing a transformation obtained through calibration-->
-<!--Calibration generated at 19:17:24, 15/03/2019 -->
+<!--Calibration generated at 19:26:05, 15/03/2019 -->
 <!--This file was written automatically using the "rosrun smobex_calibration store_calibration" command. -->
-<xacro:property name="roll" value="0.00934253096996"/>
-<xacro:property name="pitch" value="0.066844248775"/>
-<xacro:property name="yaw" value="0.0175544265835"/>
-<xacro:property name="x" value="0.0898634033575"/>
-<xacro:property name="y" value="0.0386030299782"/>
-<xacro:property name="z" value="-0.00850057584549"/>
+<xacro:property name="roll" value="-0.000577203098326"/>
+<xacro:property name="pitch" value="0.0506970123345"/>
+<xacro:property name="yaw" value="0.0240205718001"/>
+<xacro:property name="x" value="0.100036583302"/>
+<xacro:property name="y" value="0.00452059994047"/>
+<xacro:property name="z" value="0.00438971972985"/>
 </robot>

Commit message: add moveit_config for fanuc+xtion and py jnt move

File: smobex_calibration/calibration/calib_vals.xacro (robot description, xacro)
@@ -2,11 +2,11 @@
 <robot xmlns:xacro="http://www.ros.org/wiki/xacro">
 <!--This xacro contains six xacro propperties representing a transformation obtained through calibration-->
-<!--Calibration generated at 19:26:05, 15/03/2019 -->
+<!--Calibration generated at 09:45:06, 18/03/2019 -->
 <!--This file was written automatically using the "rosrun smobex_calibration store_calibration" command. -->
-<xacro:property name="roll" value="-0.000577203098326"/>
-<xacro:property name="pitch" value="0.0506970123345"/>
-<xacro:property name="yaw" value="0.0240205718001"/>
-<xacro:property name="x" value="0.100036583302"/>
-<xacro:property name="y" value="0.00452059994047"/>
-<xacro:property name="z" value="0.00438971972985"/>
+<xacro:property name="roll" value="0.0108383046183"/>
+<xacro:property name="pitch" value="0.0678197638855"/>
+<xacro:property name="yaw" value="0.00317524621708"/>
+<xacro:property name="x" value="0.104268080023"/>
+<xacro:property name="y" value="-0.00786476924183"/>
+<xacro:property name="z" value="0.0191097214271"/>
 </robot>

Commit message: added random poses generator

File: smobex_calibration/calibration/calib_vals.xacro (robot description, xacro)
@@ -2,11 +2,11 @@
 <robot xmlns:xacro="http://www.ros.org/wiki/xacro">
 <!--This xacro contains six xacro propperties representing a transformation obtained through calibration-->
-<!--Calibration generated at 09:45:06, 18/03/2019 -->
+<!--Calibration generated at 17:20:59, 25/03/2019 -->
 <!--This file was written automatically using the "rosrun smobex_calibration store_calibration" command. -->
-<xacro:property name="roll" value="0.0108383046183"/>
-<xacro:property name="pitch" value="0.0678197638855"/>
-<xacro:property name="yaw" value="0.00317524621708"/>
-<xacro:property name="x" value="0.104268080023"/>
-<xacro:property name="y" value="-0.00786476924183"/>
-<xacro:property name="z" value="0.0191097214271"/>
+<xacro:property name="roll" value="0.0154379198854"/>
+<xacro:property name="pitch" value="0.0578364065282"/>
+<xacro:property name="yaw" value="-0.002961655231"/>
+<xacro:property name="x" value="0.0815268892994"/>
+<xacro:property name="y" value="-0.00113047071967"/>
+<xacro:property name="z" value="0.0145647357262"/>
 </robot>

Commit message: readme and values update

File: smobex_calibration/calibration/calib_vals.xacro (robot description, xacro)
@@ -2,11 +2,11 @@
 <robot xmlns:xacro="http://www.ros.org/wiki/xacro">
 <!--This xacro contains six xacro propperties representing a transformation obtained through calibration-->
-<!--Calibration generated at 17:20:59, 25/03/2019 -->
+<!--Calibration generated at 11:17:35, 03/04/2019 -->
 <!--This file was written automatically using the "rosrun smobex_calibration store_calibration" command. -->
-<xacro:property name="roll" value="0.0154379198854"/>
-<xacro:property name="pitch" value="0.0578364065282"/>
-<xacro:property name="yaw" value="-0.002961655231"/>
-<xacro:property name="x" value="0.0815268892994"/>
-<xacro:property name="y" value="-0.00113047071967"/>
-<xacro:property name="z" value="0.0145647357262"/>
+<xacro:property name="roll" value="0.0795325235673"/>
+<xacro:property name="pitch" value="0.090829694837"/>
+<xacro:property name="yaw" value="-0.000214995142099"/>
+<xacro:property name="x" value="0.0944091689743"/>
+<xacro:property name="y" value="0.00426136365872"/>
+<xacro:property name="z" value="0.00128318784342"/>
 </robot>

Commit message: implemented ray points generation (eval too slow)

File: smobex_calibration/calibration/calib_vals.xacro (robot description, xacro)
@@ -2,11 +2,11 @@
 <robot xmlns:xacro="http://www.ros.org/wiki/xacro">
 <!--This xacro contains six xacro propperties representing a transformation obtained through calibration-->
-<!--Calibration generated at 11:17:35, 03/04/2019 -->
+<!--Calibration generated at 16:01:34, 10/04/2019 -->
 <!--This file was written automatically using the "rosrun smobex_calibration store_calibration" command. -->
-<xacro:property name="roll" value="0.0795325235673"/>
-<xacro:property name="pitch" value="0.090829694837"/>
-<xacro:property name="yaw" value="-0.000214995142099"/>
-<xacro:property name="x" value="0.0944091689743"/>
-<xacro:property name="y" value="0.00426136365872"/>
-<xacro:property name="z" value="0.00128318784342"/>
+<xacro:property name="roll" value="0.0545855936749"/>
+<xacro:property name="pitch" value="0.0968693323016"/>
+<xacro:property name="yaw" value="0.00696298091631"/>
+<xacro:property name="x" value="0.0685608471825"/>
+<xacro:property name="y" value="-0.0044062540072"/>
+<xacro:property name="z" value="0.000766099861553"/>
 </robot>

Commit message: addeed colored arrow evaluations

File: smobex_calibration/calibration/calib_vals.xacro (robot description, xacro)
@@ -2,11 +2,11 @@
 <robot xmlns:xacro="http://www.ros.org/wiki/xacro">
 <!--This xacro contains six xacro propperties representing a transformation obtained through calibration-->
-<!--Calibration generated at 16:01:34, 10/04/2019 -->
+<!--Calibration generated at 09:36:19, 23/04/2019 -->
 <!--This file was written automatically using the "rosrun smobex_calibration store_calibration" command. -->
-<xacro:property name="roll" value="0.0545855936749"/>
-<xacro:property name="pitch" value="0.0968693323016"/>
-<xacro:property name="yaw" value="0.00696298091631"/>
-<xacro:property name="x" value="0.0685608471825"/>
-<xacro:property name="y" value="-0.0044062540072"/>
-<xacro:property name="z" value="0.000766099861553"/>
+<xacro:property name="roll" value="0.0756132471821"/>
+<xacro:property name="pitch" value="0.097417323045"/>
+<xacro:property name="yaw" value="0.00832109238411"/>
+<xacro:property name="x" value="0.0688404147861"/>
+<xacro:property name="y" value="-0.00188796578965"/>
+<xacro:property name="z" value="0.00881333507887"/>
 </robot>

Commit message: Efforts to solve "stretched arm" issue didn't work

File: smobex_calibration/calibration/calib_vals.xacro (robot description, xacro)
@@ -2,11 +2,11 @@
 <robot xmlns:xacro="http://www.ros.org/wiki/xacro">
 <!--This xacro contains six xacro propperties representing a transformation obtained through calibration-->
-<!--Calibration generated at 09:36:19, 23/04/2019 -->
+<!--Calibration generated at 16:01:52, 16/05/2019 -->
 <!--This file was written automatically using the "rosrun smobex_calibration store_calibration" command. -->
-<xacro:property name="roll" value="0.0756132471821"/>
-<xacro:property name="pitch" value="0.097417323045"/>
-<xacro:property name="yaw" value="0.00832109238411"/>
-<xacro:property name="x" value="0.0688404147861"/>
-<xacro:property name="y" value="-0.00188796578965"/>
-<xacro:property name="z" value="0.00881333507887"/>
+<xacro:property name="roll" value="0.0589793302573"/>
+<xacro:property name="pitch" value="0.0587510718812"/>
+<xacro:property name="yaw" value="0.0320912427487"/>
+<xacro:property name="x" value="0.172357173584"/>
+<xacro:property name="y" value="-0.0160552895454"/>
+<xacro:property name="z" value="0.0781311644206"/>
 </robot>

Commit message: some more tries

File: smobex_calibration/calibration/calib_vals.xacro (robot description, xacro)
@@ -1,12 +1,12 @@
 <?xml version="1.0"?>
 <robot xmlns:xacro="http://www.ros.org/wiki/xacro">
-<!--This xacro contains six xacro propperties representing a transformation obtained through calibration-->
-<!--Calibration generated at 16:01:52, 16/05/2019 -->
-<!--This file was written automatically using the "rosrun smobex_calibration store_calibration" command. -->
-<xacro:property name="roll" value="0.0589793302573"/>
-<xacro:property name="pitch" value="0.0587510718812"/>
-<xacro:property name="yaw" value="0.0320912427487"/>
-<xacro:property name="x" value="0.172357173584"/>
-<xacro:property name="y" value="-0.0160552895454"/>
-<xacro:property name="z" value="0.0781311644206"/>
+    <!--This xacro contains six xacro propperties representing a transformation obtained through calibration-->
+    <!--Calibration generated at 14:11:10, 22/05/2019 -->
+    <!--This file was written automatically using the "rosrun smobex_calibration store_calibration" command. -->
+    <xacro:property name="roll" value="0.0705631628597"/>
+    <xacro:property name="pitch" value="0.0800765806867"/>
+    <xacro:property name="yaw" value="0.00297065394398"/>
+    <xacro:property name="x" value="0.108546244873"/>
+    <xacro:property name="y" value="0.00786073211074"/>
+    <xacro:property name="z" value="0.00438827570731"/>
 </robot>

Commit message: only to store changes

File: smobex_calibration/calibration/calib_vals.xacro (robot description, xacro)
@@ -1,12 +1,12 @@
 <?xml version="1.0"?>
 <robot xmlns:xacro="http://www.ros.org/wiki/xacro">
-    <!--This xacro contains six xacro propperties representing a transformation obtained through calibration-->
-    <!--Calibration generated at 14:11:10, 22/05/2019 -->
-    <!--This file was written automatically using the "rosrun smobex_calibration store_calibration" command. -->
-    <xacro:property name="roll" value="0.0705631628597"/>
-    <xacro:property name="pitch" value="0.0800765806867"/>
-    <xacro:property name="yaw" value="0.00297065394398"/>
-    <xacro:property name="x" value="0.108546244873"/>
-    <xacro:property name="y" value="0.00786073211074"/>
-    <xacro:property name="z" value="0.00438827570731"/>
+<!--This xacro contains six xacro propperties representing a transformation obtained through calibration-->
+<!--Calibration generated at 12:29:06, 04/06/2019 -->
+<!--This file was written automatically using the "rosrun smobex_calibration store_calibration" command. -->
+<xacro:property name="roll" value="0.064741402057"/>
+<xacro:property name="pitch" value="0.0707882937096"/>
+<xacro:property name="yaw" value="0.0197628001792"/>
+<xacro:property name="x" value="0.0703526838451"/>
+<xacro:property name="y" value="0.00681133639206"/>
+<xacro:property name="z" value="0.00286629164793"/>
 </robot>

Commit message: nothing major

File: smobex_calibration/calibration/calib_vals.xacro (robot description, xacro)
@@ -2,11 +2,11 @@
 <robot xmlns:xacro="http://www.ros.org/wiki/xacro">
 <!--This xacro contains six xacro propperties representing a transformation obtained through calibration-->
-<!--Calibration generated at 12:29:06, 04/06/2019 -->
+<!--Calibration generated at 18:14:47, 16/06/2019 -->
 <!--This file was written automatically using the "rosrun smobex_calibration store_calibration" command. -->
-<xacro:property name="roll" value="0.064741402057"/>
-<xacro:property name="pitch" value="0.0707882937096"/>
-<xacro:property name="yaw" value="0.0197628001792"/>
-<xacro:property name="x" value="0.0703526838451"/>
-<xacro:property name="y" value="0.00681133639206"/>
-<xacro:property name="z" value="0.00286629164793"/>
+<xacro:property name="roll" value="0.0758974861637"/>
+<xacro:property name="pitch" value="0.087935712976"/>
+<xacro:property name="yaw" value="0.0177853040494"/>
+<xacro:property name="x" value="0.0710365269196"/>
+<xacro:property name="y" value="-0.00810728094062"/>
+<xacro:property name="z" value="0.00995643533705"/>
 </robot>
